Commit message: Mode 1 V.1

File: robot/visual/my-robot.xacro (robot description, xacro)
@@ -10,4 +10,5 @@
   <link name="link_1">
     <visual>
+    <origin xyz="0 0 0" rpy="0 0 ${3.14/2}"/>
       <geometry>
         <mesh filename="file:///$(find fun4)/meshes/link_1.stl"/>
@@ -28,5 +29,5 @@
   <link name="link_2">
     <visual>
-      <origin xyz="0.0 0.0 0.0" rpy="0 0 ${-3.14/2}"/>
+      <origin xyz="0.0 0.0 0.0" rpy="0 0 0"/>
       <geometry>
         <mesh filename="file:///$(find fun4)/meshes/link_2.stl"/>
@@ -37,5 +38,5 @@
     <parent link="link_1"/>
     <child link="link_2"/>
-    <origin xyz="0.0 -0.12 0.0" rpy="${-3.14/2} 0 0"/>
+    <origin xyz="0.12 0.0 0.0" rpy="0 ${-3.14/2} 0"/>
     <axis xyz="0 0 1"/>
     <limit
@@ -47,5 +48,5 @@
   <link name="link_3">
     <visual>
-      <origin xyz="0.0 0.0 0.0" rpy="0 0 ${-3.14/2}"/>
+      <origin xyz="0.0 0.0 0.0" rpy="0 0 0"/>
       <geometry>
         <mesh filename="file:///$(find fun4)/meshes/link_3.stl"/>
@@ -56,5 +57,5 @@
     <parent link="link_2"/>
     <child link="link_3"/>
-    <origin xyz="0.0 -0.25 0.1" rpy="0 0 0"/>
+    <origin xyz="0.25 0 0.1 " rpy="0 0 0"/>
     <axis xyz="0 0 1"/>
     <limit
@@ -75,5 +76,5 @@
     <parent link="link_3"/>
     <child link="end_effector"/>
-    <origin xyz="0.0 -0.28 0.0" rpy="${3.14/2} 0 0"/>
+    <origin xyz="0.28 0.0 0.0" rpy="0 ${3.14/2} 0"/>
   </joint>
 </robot>
